File: lolly_pcb/mini_lolly_pcb/mini_lolly_pcb.kicad_sch (KiCad schematic)
At the start: 64 parts

Commit message: add tracks and vias
Connections:
- net at D1.2 (DOUT): now also D2.4 (DIN)

Commit message: somewhat working version
Parts:
- removed D64: WS2812B, LED_SMD:LED_WS2812B_PLCC4_5.0x5.0mm_P3.2mm, symbol LED:WS2812B
Connections:
- net at D62.2 (DOUT): no longer D63.4 (DIN)

Commit message: rotate outermost leds for space
Parts:
- added J1: Conn_01x01, symbol Connector_Generic:Conn_01x01
- added J2: Conn_01x01_Pin, symbol Connector:Conn_01x01_Pin
Connections:
- net at D62.2 (DOUT): now also D63.4 (DIN)
